File: 6cm_tvtr_RF.brd (EAGLE design)
At the start: 148 x 53 mm, 14 parts

Commit message: matching
Parts:
- added U$5: 5_32_BP_ISOL, microstrip:532_R4003C_508_3EC
- added U$6: 5_7_GHZ_BP_ISOL, microstrip:576_R403C_508_5TH
- moved U$2 14.0 mm to (65.7, 14.5)
- moved U$4 4.58 mm to (22.9, 24.1)
- moved C3 4.58 mm to (10.8, 7.62)
- moved L1 4.58 mm to (6.35, 9.53)
- moved U$3 4.58 mm to (15.2, 7.62)
- moved C1 4.58 mm to (5.08, 7.62)
- moved C2 4.58 mm to (7.62, 7.62)
- moved L2 4.58 mm to (8.89, 9.53)
- moved R1 4.58 mm to (17.8, 10.8)
- moved C4 4.58 mm to (17.8, 16.5)
- moved C5 4.58 mm to (26.0, 27.3)
- moved C6 4.58 mm to (26.0, 24.8)
- moved R2 4.58 mm to (23.5, 26.0)
- moved U$1 4.58 mm to (20.3, 7.62)
Connections:
- new net N$6: U$2.G, U$5.P$2
- net GND: now also U$2.S1, U$2.S2
- net N$5: now also U$5.P$1
Other:
- board size 148 x 53 mm -> 102.3 x 101.3 mm
Changed lines of the file:
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@@
 <setting verticaltext="up"/>
 </settings>
-<grid distance="0.05" unitdist="inch" unit="mm" style="lines" multiple="1" display="no" altdistance="0.025" altunitdist="inch" altunit="inch"/>
+<grid distance="0.05" unitdist="inch" unit="mm" style="lines" multiple="1" display="no" altdistance="0" altunitdist="inch" altunit="inch"/>
 <layers>
 <layer number="1" name="Top" color="4" fill="1" visible="yes" active="yes"/>
@@
 <board>
 <plain>
-<wire x1="0" y1="0" x2="148" y2="0" width="0" layer="20"/>
-<wire x1="148" y1="0" x2="148" y2="53" width="0" layer="20"/>
-<wire x1="148" y1="53" x2="0" y2="53" width="0" layer="20"/>
-<wire x1="0" y1="53" x2="0" y2="0" width="0" layer="20"/>
+<wire x1="0" y1="0" x2="102.28" y2="0" width="0" layer="20"/>
+<wire x1="102.28" y1="0" x2="102.28" y2="101.26" width="0" layer="20"/>
+<wire x1="102.28" y1="101.26" x2="0" y2="101.26" width="0" layer="20"/>
+<wire x1="0" y1="101.26" x2="0" y2="0" width="0" layer="20"/>
 </plain>
 <attributes>
@@
 </autorouter>
 <elements>
-<element name="U$1" library="RF" package="CEL_FET" value="CE3512K2" x="22.86" y="11.43"/>
-<element name="U$2" library="RF" package="CEL_FET" value="CE3512K2" x="52.07" y="11.43"/>
-<element name="C1" library="rcl" package="C0603K" value="" x="7.62" y="11.43"/>
-<element name="C2" library="rcl" package="C0603K" value="" x="10.16" y="11.43"/>
-<element name="C3" library="rcl" package="C0603K" value="" x="13.335" y="11.43"/>
-<element name="C4" library="rcl" package="C0603K" value="" x="20.32" y="20.32" rot="R270"/>
-<element name="L1" library="inductors" package="0603" value="0603" x="8.89" y="13.335" rot="R270"/>
-<element name="L2" library="inductors" package="0603" value="0603" x="11.43" y="13.335" rot="R270"/>
-<element name="R1" library="resistor" package="R0603" value="" x="20.32" y="14.605" rot="R90"/>
-<element name="U$3" library="RF" package="HAIRPIN" value="HAIRPIN" x="17.78" y="11.43"/>
-<element name="R2" library="resistor" package="R0603" value="" x="26.035" y="29.845" rot="R90"/>
-<element name="C5" library="rcl" package="C0603K" value="" x="28.575" y="31.115" rot="R180"/>
-<element name="C6" library="rcl" package="C0603K" value="" x="28.575" y="28.575" rot="R180"/>
-<element name="U$4" library="RF" package="FLAKE_576" value="57_FLAKE" x="25.4" y="27.94" rot="R180"/>
+<element name="U$1" library="RF" package="CEL_FET" value="CE3512K2" x="20.32" y="7.62"/>
+<element name="U$2" library="RF" package="CEL_FET" value="CE3512K2" x="65.714803125" y="14.526734375"/>
+<element name="C1" library="rcl" package="C0603K" value="" x="5.08" y="7.62"/>
+<element name="C2" library="rcl" package="C0603K" value="" x="7.62" y="7.62"/>
+<element name="C3" library="rcl" package="C0603K" value="" x="10.795" y="7.62"/>
+<element name="C4" library="rcl" package="C0603K" value="" x="17.78" y="16.51" rot="R270"/>
+<element name="L1" library="inductors" package="0603" value="0603" x="6.35" y="9.525" rot="R270"/>
+<element name="L2" library="inductors" package="0603" value="0603" x="8.89" y="9.525" rot="R270"/>
+<element name="R1" library="resistor" package="R0603" value="" x="17.78" y="10.795" rot="R90"/>
+<element name="U$3" library="RF" package="HAIRPIN" value="HAIRPIN" x="15.24" y="7.62"/>
+<element name="R2" library="resistor" package="R0603" value="" x="23.495" y="26.035" rot="R90"/>
+<element name="C5" library="rcl" package="C0603K" value="" x="26.035" y="27.305" rot="R180"/>
+<element name="C6" library="rcl" package="C0603K" value="" x="26.035" y="24.765" rot="R180"/>
+<element name="U$4" library="RF" package="FLAKE_576" value="57_FLAKE" x="22.86" y="24.13" rot="R180"/>
+<element name="U$5" library="microstrip" package="532_R4003C_508_3EC" value="5_32_BP_ISOL" x="59.098078125" y="13.63096875" rot="R180"/>
+<element name="U$6" library="microstrip" package="576_R403C_508_5TH" value="5_7_GHZ_BP_ISOL" x="60.96" y="43.18" rot="R180"/>
 </elements>
 <signals>
@@
 <contactref element="L1" pad="P$2"/>
 <contactref element="C2" pad="1"/>
-<wire x1="9.285" y1="11.43" x2="8.89" y2="11.43" width="1.016" layer="1"/>
-<wire x1="8.89" y1="11.43" x2="8.495" y2="11.43" width="1.016" layer="1"/>
-<wire x1="8.89" y1="12.635" x2="8.89" y2="11.43" width="1.016" layer="1"/>
+<wire x1="6.745" y1="7.62" x2="6.35" y2="7.62" width="1.016" layer="1"/>
+<wire x1="6.35" y1="7.62" x2="5.955" y2="7.62" width="1.016" layer="1"/>
+<wire x1="6.35" y1="8.825" x2="6.35" y2="7.62" width="1.016" layer="1"/>
 </signal>
 <signal name="N$2">
@@
 <contactref element="C3" pad="1"/>
 <contactref element="L2" pad="P$2"/>
-<wire x1="12.46" y1="11.43" x2="11.43" y2="11.43" width="1.016" layer="1"/>
-<wire x1="11.43" y1="11.43" x2="11.035" y2="11.43" width="1.016" layer="1"/>
-<wire x1="11.43" y1="12.635" x2="11.43" y2="11.43" width="1.016" layer="1"/>
+<wire x1="9.92" y1="7.62" x2="8.89" y2="7.62" width="1.016" layer="1"/>
+<wire x1="8.89" y1="7.62" x2="8.495" y2="7.62" width="1.016" layer="1"/>
+<wire x1="8.89" y1="8.825" x2="8.89" y2="7.62" width="1.016" layer="1"/>
 </signal>
 <signal name="N$3">
 <contactref element="C3" pad="2"/>
 <contactref element="U$3" pad="P$1"/>
-<wire x1="15.875" y1="11.43" x2="14.21" y2="11.43" width="1.016" layer="1"/>
+<wire x1="13.335" y1="7.62" x2="11.67" y2="7.62" width="1.016" layer="1"/>
 </signal>
 <signal name="N$4">
@@
 <contactref element="R1" pad="1"/>
 <contactref element="U$3" pad="P$2"/>
-<wire x1="21.37" y1="11.43" x2="20.32" y2="11.43" width="1.016" layer="1"/>
-<wire x1="20.32" y1="11.43" x2="19.685" y2="11.43" width="1.016" layer="1"/>
-<wire x1="20.32" y1="13.755" x2="20.32" y2="11.43" width="0.4064" layer="1"/>
+<wire x1="18.83" y1="7.62" x2="17.78" y2="7.62" width="1.016" layer="1"/>
+<wire x1="17.78" y1="7.62" x2="17.145" y2="7.62" width="1.016" layer="1"/>
+<wire x1="17.78" y1="9.945" x2="17.78" y2="7.62" width="0.4064" layer="1"/>
 </signal>
 <signal name="GND" airwireshidden="yes">
@@
 <contactref element="C6" pad="1"/>
 <contactref element="C5" pad="1"/>
-<wire x1="11.43" y1="14.035" x2="8.89" y2="14.035" width="0" layer="19" extent="1-1"/>
-<wire x1="20.32" y1="21.195" x2="11.43" y2="14.035" width="0" layer="19" extent="1-1"/>
-<wire x1="22.86" y1="12.92" x2="20.32" y2="21.195" width="0" layer="19" extent="1-1"/>
-<wire x1="22.86" y1="9.94" x2="22.86" y2="12.92" width="0" layer="19" extent="1-1"/>
-<wire x1="29.45" y1="28.575" x2="20.32" y2="21.195" width="0" layer="19" extent="1-1"/>
-<wire x1="29.45" y1="31.115" x2="29.45" y2="28.575" width="0" layer="19" extent="1-1"/>
+<contactref element="U$2" pad="S1"/>
+<contactref element="U$2" pad="S2"/>
+<wire x1="65.714803125" y1="13.036734375" x2="65.714803125" y2="16.016734375" width="0" layer="19" extent="1-1"/>
+<wire x1="26.91" y1="24.765" x2="65.714803125" y2="16.016734375" width="0" layer="19" extent="1-1"/>
+<wire x1="26.91" y1="27.305" x2="26.91" y2="24.765" width="0" layer="19" extent="1-1"/>
+<wire x1="17.78" y1="17.385" x2="26.91" y2="24.765" width="0" layer="19" extent="1-1"/>
+<wire x1="20.32" y1="9.11" x2="17.78" y2="17.385" width="0" layer="19" extent="1-1"/>
+<wire x1="20.32" y1="6.13" x2="20.32" y2="9.11" width="0" layer="19" extent="1-1"/>
+<wire x1="8.89" y1="10.225" x2="17.78" y2="17.385" width="0" layer="19" extent="1-1"/>
+<wire x1="6.35" y1="10.225" x2="8.89" y2="10.225" width="0" layer="19" extent="1-1"/>
 </signal>
 <signal name="D1">
 <contactref element="R2" pad="2"/>
 <contactref element="C5" pad="2"/>
-<via x="26.035" y="33.655" extent="1-16" drill="1.2"/>
-<wire x1="26.035" y1="30.695" x2="26.035" y2="33.655" width="0" layer="19" extent="1-1"/>
-<wire x1="27.7" y1="31.115" x2="26.035" y2="30.695" width="0" layer="19" extent="1-1"/>
+<via x="23.495" y="29.845" extent="1-16" drill="1.2"/>
+<wire x1="23.495" y1="26.885" x2="23.495" y2="29.845" width="0" layer="19" extent="1-1"/>
+<wire x1="25.16" y1="27.305" x2="23.495" y2="26.885" width="0" layer="19" extent="1-1"/>
 </signal>
 <signal name="N$5">
@@
 <contactref element="R2" pad="1"/>
 <contactref element="C6" pad="2"/>
-<wire x1="24.35" y1="11.43" x2="26.035" y2="11.43" width="1.016" layer="1"/>
-<wire x1="26.035" y1="11.43" x2="26.035" y2="28.575" width="0.3048" layer="1"/>
+<wire x1="21.81" y1="7.62" x2="23.495" y2="7.62" width="1.016" layer="1"/>
+<wire x1="23.495" y1="7.62" x2="23.495" y2="24.765" width="0.3048" layer="1"/>
 <contactref element="U$4" pad="P$1"/>
-<wire x1="26.035" y1="28.575" x2="26.035" y2="28.995" width="0" layer="19" extent="1-1"/>
-<wire x1="25.4" y1="27.94" x2="26.035" y2="28.575" width="0" layer="19" extent="1-1"/>
-<wire x1="27.7" y1="28.575" x2="26.035" y2="28.575" width="0" layer="19" extent="1-1"/>
+<contactref element="U$5" pad="P$1"/>
+<wire x1="23.495" y1="24.765" x2="23.495" y2="25.185" width="0" layer="19" extent="1-1"/>
+<wire x1="22.86" y1="24.13" x2="23.495" y2="24.765" width="0" layer="19" extent="1-1"/>
+<wire x1="25.16" y1="24.765" x2="23.495" y2="24.765" width="0" layer="19" extent="1-1"/>
+<wire x1="23.607784375" y1="7.61810625" x2="23.495" y2="7.62" width="0" layer="19" extent="1-1"/>
 </signal>
 <signal name="G1">
 <contactref element="C4" pad="2"/>
 <contactref element="R1" pad="2"/>
-<via x="20.32" y="17.78" extent="1-16" drill="1.2"/>
-<wire x1="20.32" y1="19.445" x2="20.32" y2="17.78" width="0" layer="19" extent="1-1"/>
-<wire x1="20.32" y1="15.455" x2="20.32" y2="19.445" width="0" layer="19" extent="1-1"/>
+<via x="17.78" y="13.97" extent="1-16" drill="1.2"/>
+<wire x1="17.78" y1="15.635" x2="17.78" y2="13.97" width="0" layer="19" extent="1-1"/>
+<wire x1="17.78" y1="11.645" x2="17.78" y2="15.635" width="0" layer="19" extent="1-1"/>
+</signal>
+<signal name="N$6">
+<contactref element="U$5" pad="P$2"/>
+<contactref element="U$2" pad="G"/>
+<wire x1="61.83305" y1="14.531596875" x2="64.224803125" y2="14.526734375" width="0" layer="19" extent="1-1"/>
 </signal>
 </signals>
