File: 6cm_tvtr_RF.sch (EAGLE design)
At the start: 14 parts

Commit message: matching
Parts:
- added U$5: 5_32_BP_ISOL, microstrip:5_32_BP_ISOL
- added U$6: 5_7_GHZ_BP_ISOL, microstrip:5_7_GHZ_BP_ISOL
Connections:
- new net N$6: U$2.G, U$5.P$2
- net GND: now also U$2.S
- net N$5: now also U$5.P$1
Changed lines of the file:
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@@
 <part name="GND5" library="supply1" deviceset="GND" device=""/>
 <part name="U$4" library="RF" deviceset="57_FLAKE" device=""/>
+<part name="U$5" library="microstrip" deviceset="5_32_BP_ISOL" device=""/>
+<part name="GND6" library="supply1" deviceset="GND" device=""/>
+<part name="U$6" library="microstrip" deviceset="5_7_GHZ_BP_ISOL" device=""/>
 </parts>
 <sheets>
@@
 <instances>
 <instance part="U$1" gate="G$1" x="43.18" y="38.1"/>
-<instance part="U$2" gate="G$1" x="116.84" y="35.56"/>
+<instance part="U$2" gate="G$1" x="116.84" y="43.18"/>
 <instance part="C1" gate="G$1" x="-60.96" y="38.1" rot="R90"/>
 <instance part="C2" gate="G$1" x="-38.1" y="38.1" rot="R90"/>
@@
 <instance part="GND5" gate="1" x="63.5" y="60.96"/>
 <instance part="U$4" gate="G$1" x="45.72" y="53.34" rot="R180"/>
+<instance part="U$5" gate="G$1" x="76.2" y="43.18"/>
+<instance part="GND6" gate="1" x="119.38" y="17.78"/>
+<instance part="U$6" gate="G$1" x="175.26" y="45.72"/>
 </instances>
 <busses>
@@
 <junction x="63.5" y="66.04"/>
 </segment>
+<segment>
+<pinref part="GND6" gate="1" pin="GND"/>
+<pinref part="U$2" gate="G$1" pin="S"/>
+<wire x1="119.38" y1="20.32" x2="119.38" y2="38.1" width="0.1524" layer="91"/>
+</segment>
 </net>
 <net name="D1" class="0">
@@
 <pinref part="U$4" gate="G$1" pin="P$1"/>
 <junction x="45.72" y="53.34"/>
+<pinref part="U$5" gate="G$1" pin="P$1"/>
+<wire x1="68.58" y1="43.18" x2="45.72" y2="43.18" width="0.1524" layer="91"/>
 </segment>
 </net>
@@
 </segment>
 </net>
+<net name="N$6" class="0">
+<segment>
+<pinref part="U$5" gate="G$1" pin="P$2"/>
+<pinref part="U$2" gate="G$1" pin="G"/>
+<wire x1="83.82" y1="43.18" x2="114.3" y2="43.18" width="0.1524" layer="91"/>
+</segment>
+</net>

Commit message: Output Match
Parts:
- added C7: (no value), rcl:C-EUC0603K
- added U$7: Q1_INPUT, microstrip:Q1_INPUT
- added U$8: MDB-73H+, microstrip:MDB-73H+
Connections:
- new net N$10: U$2.D
- new net N$11: U$6.P$1, U$8.RF
- new net N$7: U$2.G, U$7.OUT
- new net N$9: C7.1, U$8.LO
- net GND: now also U$8.GND
- net N$6: now also U$7.IN; no longer U$2.G
Other:
- moved on the sheet: U$6
Changed lines of the file:
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@@
 <part name="GND6" library="supply1" deviceset="GND" device=""/>
 <part name="U$6" library="microstrip" deviceset="5_7_GHZ_BP_ISOL" device=""/>
+<part name="U$7" library="microstrip" deviceset="Q1_INPUT" device=""/>
+<part name="U$8" library="microstrip" deviceset="MDB-73H+" device=""/>
+<part name="GND7" library="supply1" deviceset="GND" device=""/>
+<part name="C7" library="rcl" deviceset="C-EU" device="C0603K"/>
 </parts>
 <sheets>
@@
 <instance part="U$5" gate="G$1" x="76.2" y="43.18"/>
 <instance part="GND6" gate="1" x="119.38" y="17.78"/>
-<instance part="U$6" gate="G$1" x="175.26" y="45.72"/>
+<instance part="U$6" gate="G$1" x="175.26" y="55.88"/>
+<instance part="U$7" gate="G$1" x="93.98" y="43.18"/>
+<instance part="U$8" gate="G$1" x="147.32" y="53.34"/>
+<instance part="GND7" gate="1" x="152.4" y="38.1"/>
+<instance part="C7" gate="G$1" x="132.08" y="55.88" rot="R270"/>
 </instances>
 <busses>
@@
 <wire x1="119.38" y1="20.32" x2="119.38" y2="38.1" width="0.1524" layer="91"/>
 </segment>
+<segment>
+<pinref part="U$8" gate="G$1" pin="GND"/>
+<wire x1="152.4" y1="43.18" x2="152.4" y2="40.64" width="0.1524" layer="91"/>
+<pinref part="GND7" gate="1" pin="GND"/>
+</segment>
 </net>
 <net name="D1" class="0">
@@
 <segment>
 <pinref part="U$5" gate="G$1" pin="P$2"/>
-<pinref part="U$2" gate="G$1" pin="G"/>
-<wire x1="83.82" y1="43.18" x2="114.3" y2="43.18" width="0.1524" layer="91"/>
+<pinref part="U$7" gate="G$1" pin="IN"/>
+<wire x1="83.82" y1="43.18" x2="91.44" y2="43.18" width="0.1524" layer="91"/>
 </segment>
 </net>
+<net name="N$7" class="0">
+<segment>
+<pinref part="U$7" gate="G$1" pin="OUT"/>
+<pinref part="U$2" gate="G$1" pin="G"/>
+<wire x1="104.14" y1="43.18" x2="114.3" y2="43.18" width="0.1524" layer="91"/>
+</segment>
+</net>
+<net name="N$9" class="0">
+<segment>
+<pinref part="U$8" gate="G$1" pin="LO"/>
+<wire x1="139.7" y1="55.88" x2="134.62" y2="55.88" width="0.1524" layer="91"/>
+<pinref part="C7" gate="G$1" pin="1"/>
+</segment>
+</net>
+<net name="N$10" class="0">
+<segment>
+<pinref part="U$2" gate="G$1" pin="D"/>
+<wire x1="119.38" y1="48.26" x2="119.38" y2="55.88" width="0.1524" layer="91"/>
+</segment>
+</net>
+<net name="N$11" class="0">
+<segment>
+<pinref part="U$8" gate="G$1" pin="RF"/>
+<pinref part="U$6" gate="G$1" pin="P$1"/>
+<wire x1="157.48" y1="55.88" x2="167.64" y2="55.88" width="0.1524" layer="91"/>
+</segment>
+</net>

Commit message: layout with GAL1+ etc
Parts:
- added C10, C8, C9: (no value), rcl:C-EUC0603K
- added L3, L4: 0603, inductors:0603
- added R3, R4: (no value), resistor:R-EU_R0603
- U$1: value CE3512K2 -> GALI39+; device RF:CE3512K2 -> RF:GALI39+
- U$2: value CE3512K2 -> GALI1+; device RF:CE3512K2 -> RF:GALI1+
- U$3: value HAIRPIN -> GALI39+; device RF:HAIRPIN -> RF:GALI39+
- U$4: value 57_FLAKE -> GALI1+; device RF:57_FLAKE -> RF:GALI1+
- U$7: value Q1_INPUT -> 576_WILK; device microstrip:Q1_INPUT -> RF:576_WILK
Connections:
- removed net G1: C4.2, R1.2
- new net N$12: C3.1, U$3.IN
- new net N$13: C4.2, L3.1, U$3.OUT
- new net N$14: C4.1, U$4.IN
- new net N$15: C7.2, L4.1, U$4.OUT
- new net N$16: L3.2, R3.1
- new net N$17: L4.2, R4.1
- new net N$18: C10.1, U$8.IF
- new net N$8: C1.1
- new net VCC: C2.2, R1.2
- net D1: now also C8.2, C9.2, R3.2, R4.2
- net GND: now also C2.1, C8.1, C9.1, U$1.GND, U$2.GND, U$3.GND, U$4.GND; no longer C4.1, C6.1, L1.1, L2.1, U$1.S, U$2.S
- net N$1: now also U$1.IN; no longer C2.1, L1.2
- net N$10: now also C3.2, U$7.P$2; no longer U$2.D
- net N$2: now also R2.1; no longer C2.2, C3.1
- net N$3: now also C6.2, L2.1, U$2.OUT; no longer C3.2, U$3.P$1
- net N$4: now also L1.2; no longer U$1.G, U$3.P$2
- net N$5: now also L1.1, U$1.OUT; no longer C6.2, R2.1, U$1.D, U$4.P$1
- net N$6: now also U$2.IN; no longer U$7.IN
- net N$7: now also U$6.P$2, U$7.P$1; no longer U$2.G, U$7.OUT
- net N$9: now also C6.1; no longer C7.1
Other:
- note added: "+1"
- note added: "+10"
- note added: "+5"
- note added: "+6"
- note added: "+9"
- note added: "-10"
- note added: "-2"
- note added: "-6"
- note added: "0/+6"
- moved on the sheet: C1, C2, C3, C4, C5, C6, C7, L1, L2, R1, R2, U$5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
