File: 6cm_tvtr_RF.sch (EAGLE design)
At the start: 26 parts

Commit message: misc
Parts:
- removed L2: 0603, inductors:0603
- added U$9: STUB, microstrip:STUB
- U$5: value 5_32_BP_ISOL -> 5_32_BP_ISOL532_R4350B_508_3EC; device microstrip:5_32_BP_ISOL -> microstrip:5_32_BP_ISOL532_R4350B_508_3EC
Connections:
- net N$2: now also U$9.P$2; no longer L2.2
- net N$3: now also U$9.RF_END; no longer L2.1
Other:
- moved on the sheet: C5, R2
Changed lines of the file:
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@@
 <part name="D1" library="supply1" deviceset="VCC" device="" value="D1"/>
 <part name="GND5" library="supply1" deviceset="GND" device=""/>
-<part name="U$5" library="microstrip" deviceset="5_32_BP_ISOL" device=""/>
+<part name="U$5" library="microstrip" deviceset="5_32_BP_ISOL" device="532_R4350B_508_3EC"/>
 <part name="GND6" library="supply1" deviceset="GND" device=""/>
 <part name="U$6" library="microstrip" deviceset="5_7_GHZ_BP_ISOL" device=""/>
@@
 <part name="GND7" library="supply1" deviceset="GND" device=""/>
 <part name="R1" library="resistor" deviceset="R-EU_" device="R0603"/>
-<part name="L2" library="inductors" deviceset="0603" device=""/>
 <part name="C2" library="rcl" deviceset="C-EU" device="C0603K"/>
 <part name="D2" library="supply1" deviceset="VCC" device="" value="D1"/>
@@
 <part name="GND10" library="supply1" deviceset="GND" device=""/>
 <part name="C10" library="rcl" deviceset="C-EU" device="C0603K"/>
+<part name="U$9" library="microstrip" deviceset="STUB" device=""/>
 </parts>
 <sheets>
@@
 <instance part="L1" gate="G$1" x="-22.86" y="48.26" rot="R90"/>
 <instance part="GND3" gate="1" x="15.24" y="27.94"/>
-<instance part="R2" gate="G$1" x="22.86" y="60.96" rot="R90"/>
-<instance part="C5" gate="G$1" x="30.48" y="68.58" rot="R270"/>
+<instance part="R2" gate="G$1" x="22.86" y="68.58" rot="R90"/>
+<instance part="C5" gate="G$1" x="30.48" y="76.2" rot="R270"/>
 <instance part="C6" gate="G$1" x="30.48" y="38.1" rot="R270"/>
-<instance part="D1" gate="VCC" x="22.86" y="78.74"/>
-<instance part="GND5" gate="1" x="35.56" y="63.5"/>
+<instance part="D1" gate="VCC" x="22.86" y="83.82"/>
+<instance part="GND5" gate="1" x="35.56" y="71.12"/>
 <instance part="U$5" gate="G$1" x="-7.62" y="38.1"/>
 <instance part="GND6" gate="1" x="119.38" y="17.78"/>
@@
 <instance part="GND7" gate="1" x="50.8" y="20.32"/>
 <instance part="R1" gate="G$1" x="-22.86" y="60.96" rot="R90"/>
-<instance part="L2" gate="G$1" x="22.86" y="48.26" rot="R90"/>
 <instance part="C2" gate="G$1" x="-15.24" y="68.58" rot="R270"/>
 <instance part="D2" gate="VCC" x="-22.86" y="78.74"/>
@@
 <instance part="GND10" gate="1" x="162.56" y="35.56"/>
 <instance part="C10" gate="G$1" x="43.18" y="15.24"/>
+<instance part="U$9" gate="G$1" x="22.86" y="48.26"/>
 </instances>
 <busses>
@@
 <pinref part="GND5" gate="1" pin="GND"/>
 <pinref part="C5" gate="G$1" pin="1"/>
-<wire x1="33.02" y1="68.58" x2="35.56" y2="68.58" width="0.1524" layer="91"/>
-<wire x1="35.56" y1="68.58" x2="35.56" y2="66.04" width="0.1524" layer="91"/>
+<wire x1="33.02" y1="76.2" x2="35.56" y2="76.2" width="0.1524" layer="91"/>
+<wire x1="35.56" y1="76.2" x2="35.56" y2="73.66" width="0.1524" layer="91"/>
 </segment>
 <segment>
@@
 <segment>
 <pinref part="R2" gate="G$1" pin="2"/>
-<wire x1="22.86" y1="66.04" x2="22.86" y2="68.58" width="0.1524" layer="91"/>
+<wire x1="22.86" y1="73.66" x2="22.86" y2="76.2" width="0.1524" layer="91"/>
 <pinref part="C5" gate="G$1" pin="2"/>
-<wire x1="22.86" y1="68.58" x2="25.4" y2="68.58" width="0.1524" layer="91"/>
-<wire x1="22.86" y1="68.58" x2="22.86" y2="76.2" width="0.1524" layer="91"/>
+<wire x1="22.86" y1="76.2" x2="25.4" y2="76.2" width="0.1524" layer="91"/>
+<wire x1="22.86" y1="76.2" x2="22.86" y2="81.28" width="0.1524" layer="91"/>
 <pinref part="D1" gate="VCC" pin="VCC"/>
-<junction x="22.86" y="68.58"/>
+<junction x="22.86" y="76.2"/>
 </segment>
 <segment>
@@
 <segment>
 <pinref part="R2" gate="G$1" pin="1"/>
-<pinref part="L2" gate="G$1" pin="2"/>
-<wire x1="22.86" y1="53.34" x2="22.86" y2="55.88" width="0.1524" layer="91"/>
+<wire x1="22.86" y1="58.42" x2="22.86" y2="63.5" width="0.1524" layer="91"/>
+<pinref part="U$9" gate="G$1" pin="P$2"/>
 </segment>
 </net>
@@
 <segment>
 <pinref part="U$2" gate="G$1" pin="OUT"/>
-<pinref part="L2" gate="G$1" pin="1"/>
 <wire x1="20.32" y1="38.1" x2="22.86" y2="38.1" width="0.1524" layer="91"/>
-<wire x1="22.86" y1="38.1" x2="22.86" y2="43.18" width="0.1524" layer="91"/>
+<wire x1="22.86" y1="38.1" x2="22.86" y2="40.64" width="0.1524" layer="91"/>
 <wire x1="22.86" y1="38.1" x2="25.4" y2="38.1" width="0.1524" layer="91"/>
 <pinref part="C6" gate="G$1" pin="2"/>
 <junction x="22.86" y="38.1"/>
-</segment>
-</net>
+<pinref part="U$9" gate="G$1" pin="RF_END"/>
+</segment>
+</net>
